File: Modules/DCDC_Boost(LM51571-Q1)_(3v-13v to 24v 0.3A)/DCDC_Boost(LM51571-Q1).kicad_pcb (KiCad board)
At the start: 2 copper layers, 18.6 x 13 mm, 17 parts, among them J1 Conn_01x02, J2 Conn_01x02, U1 LM51571

Commit message: Sort Out
Other:
- net class Default removed
