File: Modules/DCDC_BatCharge_(4.2v-12.6v to12.9v with [1-3cell]x4.2v)/DCDC_BATCharge(BQ24170).sch (KiCad schematic (older format))
At the start: 88 parts, among them J1 Btn_LED, J2 VIA_V_BAT, J3 VIA_GND, J4 VIA_V_Adapter, J5 VIA_V_SYS, Q1 AO3416, Q2 AO3416, Q3 AO3415, U1 BQ24170, U2 TPS61288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

Commit message: Signed-off-by: starsriver <starsriver@yahoo.com>
Parts:
- F1: value 4A -> 3.5A
- R20: value 41.2k -> 47.5k
Changed lines of the file:
@@
 P 9200 10000
 F 0 "F1" V 9397 10000 50  0000 C CNN
-F 1 "4A" V 9306 10000 50  0000 C CNN
+F 1 "3.5A" V 9306 10000 50  0000 C CNN
 F 2 "Fuse:Fuse_0603_1608Metric" V 9130 10000 50  0001 C CNN
 F 3 "~" H 9200 10000 50  0001 C CNN
@@
 P 4200 14450
 F 0 "R20" H 4130 14404 50  0000 R CNN
-F 1 "41.2k" H 4150 14500 50  0000 R CNN
+F 1 "47.5k" H 4150 14500 50  0000 R CNN
 F 2 "Resistor_SMD:R_0402_1005Metric" V 4130 14450 50  0001 C CNN
 F 3 "~" H 4200 14450 50  0001 C CNN

Commit message: update modules
Parts:
- L1: value 3.3uH CoilCraft 6030 -> 3.3uH CoilCraft 40xx; footprint Inductor_SMD:L_Coilcraft_XAL60xx_6.36x6.56mm -> Inductor_SMD:L_Coilcraft_XxL4020
- L2, L3: value 1.8uH CoilCraft 6030 -> 1.8uH CoilCraft 40xx; footprint Inductor_SMD:L_Coilcraft_XAL60xx_6.36x6.56mm -> Inductor_SMD:L_Coilcraft_XxL4020
Other:
- moved on the sheet: C1, C10, C11, C12, C13, C14, C15, C16, C17, C18, C19, C2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

Commit message: update
Parts:
- J2: value VIA_V_BAT -> VIA_V_PACK
- U1: footprint AMPF:BQ24170RGYT -> BQ24170RGYT:BQ24170RGYT; symbol AMPF:BQ24170 -> BQ24170:BQ24170
- U2, U3: footprint AMPF:TPS61288 -> TPS61288:TPS61288; symbol AMPF:TPS61288 -> TPS61288:TPS61288
Connections:
- net V_BAT renamed V_PACK
- net V_BAT_BOOST renamed V_PACK_BOOST
- net V_BAT_OUT renamed V_PACK_OUT
Other:
- moved on the sheet: Q3
Changed lines of the file:
@@
 	8950 4350 8950 4400
 Text GLabel 9250 2700 1    50   Input ~ 0
-V_BAT
+V_PACK
 $Comp
 L Device:D D1
@@
 	1500 2750 1700 2750
 $Comp
-L AMPF:TPS61288 U2
+L TPS61288:TPS61288 U2
 U 1 1 6082B738
 P 2700 2500
 F 0 "U2" H 2250 4100 50  0000 C CNN
 F 1 "TPS61288" H 2350 4000 50  0000 C CNN
-F 2 "AMPF:TPS61288" H 2650 3400 50  0001 C CNN
+F 2 "TPS61288:TPS61288" H 2650 3400 50  0001 C CNN
 F 3 "" H 2650 3400 50  0001 C CNN
 	1    2700 2500
@@
 	1500 6550 1700 6550
 $Comp
-L AMPF:TPS61288 U3
+L TPS61288:TPS61288 U3
 U 1 1 6081077F
 P 2700 6300
 F 0 "U3" H 2250 7900 50  0000 C CNN
 F 1 "TPS61288" H 2350 7800 50  0000 C CNN
-F 2 "AMPF:TPS61288" H 2650 7200 50  0001 C CNN
+F 2 "TPS61288:TPS61288" H 2650 7200 50  0001 C CNN
 F 3 "" H 2650 7200 50  0001 C CNN
 	1    2700 6300
@@
 Connection ~ 9850 3750
 $Comp
-L AMPF:BQ24170 U1
+L BQ24170:BQ24170 U1
 U 1 1 607BDACE
 P 12350 4350
 F 0 "U1" H 8900 7800 50  0000 C CNN
 F 1 "BQ24170" H 9000 7700 50  0000 C CNN
-F 2 "AMPF:BQ24170RGYT" H 12300 4450 50  0001 C CNN
+F 2 "BQ24170RGYT:BQ24170RGYT" H 12300 4450 50  0001 C CNN
 F 3 "" H 12300 4450 50  0001 C CNN
 	1    12350 4350
@@
 $EndComp
 $Comp
-L Device:Q_PMOS_GSD Q3
-U 1 1 607C2FAE
-P 14750 2450
-F 0 "Q3" H 14954 2496 50  0000 L CNN
-F 1 "AO3415" H 14954 2405 50  0000 L CNN
-F 2 "Package_TO_SOT_SMD:SOT-23" H 14950 2550 50  0001 C CNN
-F 3 "~" H 14750 2450 50  0001 C CNN
-	1    14750 2450
-	1    0    0    1
-$EndComp
-$Comp
 L Device:R R10
 U 1 1 607C1EE6
@@
 	13750 3250 14100 3250
 Wire Wire Line
-	14100 3250 14100 2450
-Wire Wire Line
-	14100 2450 14550 2450
-Wire Wire Line
-	12900 2200 14850 2200
-Wire Wire Line
-	14850 2200 14850 2250
-Text GLabel 15550 2200 2    50   Input ~ 0
-V_sys
+	14100 3250 14100 2500
 Text GLabel 15550 3050 2    50   Input ~ 0
-V_BAT
+V_PACK
 Wire Wire Line
 	15300 3050 15550 3050
-Wire Wire Line
-	14850 2200 15550 2200
-Connection ~ 14850 2200
 $Comp
 L power:GND #PWR010
@@
 	14850 2900 15550 2900
 Connection ~ 14850 3050
-Wire Wire Line
-	14850 2650 14850 2700
-Wire Wire Line
-	14850 2700 15550 2700
 Text GLabel 15550 2900 2    50   Input ~ 0
-V_BAT_OUT
-Text GLabel 15550 2700 2    50   Input ~ 0
-V_BAT_BOOST
+V_PACK_OUT
 Text GLabel 1400 6000 0    50   Input ~ 0
-V_BAT_OUT
+V_PACK_OUT
 Text GLabel 6300 6000 2    50   Input ~ 0
-V_BAT_BOOST
+V_PACK_BOOST
 $Comp
 L Graphic:SYM_Arrow_Large #SYM1
@@
 $EndComp
 Text GLabel 8300 6400 3    50   Input ~ 0
-V_BAT
+V_PACK
 $Comp
 L Connector:Conn_01x01_Female J2
@@
 P 8300 6100
 F 0 "J2" V 8250 6050 50  0000 R CNN
-F 1 "VIA_V_BAT" H 8200 5950 50  0000 R CNN
+F 1 "VIA_V_PACK" H 8200 5950 50  0000 R CNN
 F 2 "MountingHole:MountingHole_2.2mm_M2_Pad_Via" H 8300 6100 50  0001 C CNN
 F 3 "~" H 8300 6100 50  0001 C CNN
@@
 Wire Wire Line
 	8650 6300 8650 6400
+Wire Wire Line
+	14300 2200 14500 2200
+Text GLabel 14500 2200 2    50   Input ~ 0
+V_PACK_BOOST
+Text GLabel 13700 1700 1    50   Input ~ 0
+V_sys
+Wire Wire Line
+	13700 2200 13700 1700
+Wire Wire Line
+	12900 2200 13700 2200
+$Comp
+L Device:Q_PMOS_GSD Q3
+U 1 1 607C2FAE
+P 14100 2300
+F 0 "Q3" H 14304 2346 50  0000 L CNN
+F 1 "AO3415" H 14304 2255 50  0000 L CNN
+F 2 "Package_TO_SOT_SMD:SOT-23" H 14300 2400 50  0001 C CNN
+F 3 "~" H 14100 2300 50  0001 C CNN
+	1    14100 2300
+	0    1    -1   0
+$EndComp
+Wire Wire Line
+	13700 2200 13900 2200
+Connection ~ 13700 2200
 $EndSCHEMATC
