File: Modules/LDO_BatCharger(BQ21040)_(USB-4.2v 0.54A)/LDO_BatCharger(BQ21040).kicad_pcb (KiCad board)
At the start: 2 copper layers, 21.8 x 14.1 mm, 21 parts, among them J1 Conn_01x01, J2 Conn_01x01, J3 Conn_01x01, J4 Conn_01x01, J5 Conn_01x01, J6 Conn_01x01, J7 Conn_01x01, U1 BQ2970, U2 BQ21040, U3 CSD16406Q3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

Commit message: update
Connections:
- U4 pad 2: Net-(U4-Pad2) -> BAT-
- U4 pad 3: Net-(U4-Pad2) -> BAT-
Other:
- outline, holes or cut-outs redrawn
- board text added: "BAT+"
- board text added: "BAT-"
- board text added: "CHG+"
- board text added: "CHG-"
- board text added: "GND"
- board text added: "STAT"
