File: Modules/LDO_BatCharger(BQ21040)_(USB-4.2v 0.54A)/LDO_BatCharger(BQ21040).sch (KiCad schematic (older format))
At the start: 21 parts, among them J1 Conn_01x01, J2 Conn_01x01, J3 Conn_01x01, J4 Conn_01x01, J5 Conn_01x01, J6 Conn_01x01, J7 Conn_01x01, U1 BQ2970, U2 BQ21040, U3 CSD16406Q3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

Commit message: update
Connections:
- net BAT-: now also U4.2, U4.3
Changed lines of the file:
@@
 $EndComp
 Wire Wire Line
-	8950 3000 8950 2550
+	8950 3000 8950 2800
 Wire Wire Line
 	8850 3000 8950 3000
@@
 U 1 1 60927DB8
 P 8450 3200
-F 0 "U1" H 8450 3715 50  0000 C CNN
-F 1 "BQ2970" H 8450 3624 50  0000 C CNN
+F 0 "U1" H 8450 3750 50  0000 C CNN
+F 1 "BQ2970" H 8450 3650 50  0000 C CNN
 F 2 "Package_SON:WSON-6_1.5x1.5mm_P0.5mm" H 8450 3650 50  0001 C CNN
 F 3 "" H 8450 3650 50  0001 C CNN
@@
 BAT+
 Wire Wire Line
-	5900 2550 5900 3600
-Wire Wire Line
-	8950 2550 5900 2550
+	5900 2800 5900 3600
+Wire Wire Line
+	8950 2800 5900 2800
 Wire Wire Line
 	2250 3650 2250 3800
@@
 Connection ~ 7150 4050
 Connection ~ 7150 4350
+Wire Wire Line
+	7950 4100 7950 4200
+Connection ~ 7950 4200
 $EndSCHEMATC
