File: Modules/Amplifier(INA848+ADA3894-2)_(60+36dB)_(10uV-1mV)/Amplifier.sch (KiCad schematic (older format))
At the start: 59 parts, among them J1 Conn_01x04, J2 Conn_01x01_Female, J3 Conn_01x03_Female, J4 Conn_01x02_Male, J5 Conn_01x01_Female, U1 TPS7A4901DGNR, U2 TPS7A3001DGNT, U3 ina848, U4 ADA4898-2, U5 ADA4898-2

Commit message: design fix
Parts:
- C10, C17, C18, C21, C22, C9: footprint Capacitor_SMD:C_0805_2012Metric -> Capacitor_SMD:C_1206_3216Metric
Changed lines of the file:
@@
 F 0 "C18" H 7365 8146 50  0000 L CNN
 F 1 "0.1uF" H 7365 8055 50  0000 L CNN
-F 2 "Capacitor_SMD:C_0805_2012Metric" H 7288 7950 50  0001 C CNN
+F 2 "Capacitor_SMD:C_1206_3216Metric" H 7288 7950 50  0001 C CNN
 F 3 "~" H 7250 8100 50  0001 C CNN
 	1    7250 8100
@@
 F 0 "C17" H 7365 7446 50  0000 L CNN
 F 1 "0.1uF" H 7365 7355 50  0000 L CNN
-F 2 "Capacitor_SMD:C_0805_2012Metric" H 7288 7250 50  0001 C CNN
+F 2 "Capacitor_SMD:C_1206_3216Metric" H 7288 7250 50  0001 C CNN
 F 3 "~" H 7250 7400 50  0001 C CNN
 	1    7250 7400
@@
 F 0 "C21" H 8615 7446 50  0000 L CNN
 F 1 "0.1uF" H 8615 7355 50  0000 L CNN
-F 2 "Capacitor_SMD:C_0805_2012Metric" H 8538 7250 50  0001 C CNN
+F 2 "Capacitor_SMD:C_1206_3216Metric" H 8538 7250 50  0001 C CNN
 F 3 "~" H 8500 7400 50  0001 C CNN
 	1    8500 7400
@@
 F 0 "C22" H 8615 8146 50  0000 L CNN
 F 1 "0.1uF" H 8615 8055 50  0000 L CNN
-F 2 "Capacitor_SMD:C_0805_2012Metric" H 8538 7950 50  0001 C CNN
+F 2 "Capacitor_SMD:C_1206_3216Metric" H 8538 7950 50  0001 C CNN
 F 3 "~" H 8500 8100 50  0001 C CNN
 	1    8500 8100
@@
 F 0 "C10" H 4715 2746 50  0000 L CNN
 F 1 "0.1uF" H 4715 2655 50  0000 L CNN
-F 2 "Capacitor_SMD:C_0805_2012Metric" H 4638 2550 50  0001 C CNN
+F 2 "Capacitor_SMD:C_1206_3216Metric" H 4638 2550 50  0001 C CNN
 F 3 "~" H 4600 2700 50  0001 C CNN
 	1    4600 2700
@@
 F 0 "C9" H 4715 2446 50  0000 L CNN
 F 1 "0.1uF" H 4715 2355 50  0000 L CNN
-F 2 "Capacitor_SMD:C_0805_2012Metric" H 4638 2250 50  0001 C CNN
+F 2 "Capacitor_SMD:C_1206_3216Metric" H 4638 2250 50  0001 C CNN
 F 3 "~" H 4600 2400 50  0001 C CNN
 	1    4600 2400
