File: Modules/Amplifier(INA848+ADA3894-2)_(60+36dB)_(10uV-1mV)/Amplifier.kicad_pcb (KiCad board)
At the start: 4 copper layers, 81.9 x 14.8 mm, 59 parts, among them J1 Conn_01x04, J2 Conn_01x01_Female, J3 Conn_01x03_Female, J4 Conn_01x02_Male, J5 Conn_01x01_Female, U1 TPS7A4901DGNR, U2 TPS7A3001DGNT, U3 ina848, U4 ADA4898-2, U5 ADA4898-2

Commit message: design fix
Parts:
- C10, C17, C18, C21, C22, C9: footprint Capacitor_SMD:C_0805_2012Metric -> Capacitor_SMD:C_1206_3216Metric
- moved C17 0.30 mm to (111.0, 95.0)
- moved C21 0.30 mm to (100.2, 95.0)
- moved C9 0.30 mm to (88.2, 95.0)
- moved C10 0.10 mm to (88.1, 104.0)
- moved C18 0.10 mm to (106.0, 104.0)
- moved C22 0.10 mm to (95.2, 104.0)
Routing:
- net AVCC: track 27.0 -> 21.7 mm
- net AVEE: track 27.0 -> 21.7 mm

Commit message: update kicad editor version
Routing:
- net AVEE: track 21.7 -> 14.0 mm
- net AVCC: track 21.7 -> 14.5 mm
Other:
- net class Default removed
