File: Modules/WirelessPowerReceiver(BQ51013+BQ24040+BQ2971)_(5V 1A)/WirelessPower.sch (KiCad schematic (older format))
At the start: 46 parts, among them J1 Conn_01x01_Female, J2 Conn_01x01_Female, J3 Conn_01x01_Female, J4 Conn_01x01_Female, J5 BAT, J6 AC, J7 Conn_01x14, U1 BQ2971, U2 BQ51013BRHLR, U3 CSD16406Q3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

Commit message: update WirelessPower.sch (fix resistance value)
Parts:
- R2: value 15R -> 20R
- R8: value 540R -> 536R
Other:
- note added: "R2 = \n 20R -> 1.2A\n 66R -> 1A"
- note removed: "R2 = \n 15R -> 1.2A\n 66R -> 1A"
Changed lines of the file:
@@
 P 9600 3500
 F 0 "R2" H 9550 3650 50  0000 C CNN
-F 1 "15R" V 9600 3500 50  0000 C CNN
+F 1 "20R" V 9600 3500 50  0000 C CNN
 F 2 "Resistor_SMD:R_0402_1005Metric" V 9530 3500 50  0001 C CNN
 F 3 "~" H 9600 3500 50  0001 C CNN
@@
 P 2550 1350
 F 0 "R8" V 2450 1300 50  0000 C CNN
-F 1 "540R" V 2550 1350 50  0000 C CNN
+F 1 "536R" V 2550 1350 50  0000 C CNN
 F 2 "Resistor_SMD:R_0402_1005Metric" V 2480 1350 50  0001 C CNN
 F 3 "~" H 2550 1350 50  0001 C CNN
@@
 	3350 6950 3200 6950
 Text Notes 9900 2950 0    50   ~ 0
-R2 = \n 15R -> 1.2A\n 66R -> 1A
+R2 = \n 20R -> 1.2A\n 66R -> 1A
 Wire Notes Line
 	9850 2650 10550 2650
