File: Modules/DCDC_BuckBoost(TPS61088+MP1495S)_(Bat to 5V-3v3-2v5-1v5-1v2 3A)/PowerSupply.sch (KiCad schematic (older format))
At the start: 97 parts, among them J1 Conn_01x14, J10 Conn_01x01, J2 Conn_01x01, J3 Conn_01x01, J4 Conn_01x01, J5 Conn_01x01, J6 Conn_01x01, J7 Conn_01x01, J8 Conn_01x01, J9 Conn_01x01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

Commit message: update symbols in PowerSupply.sch
Parts:
- C40, C41, C42: symbol Device:CP1 -> Device:C
Changed lines of the file:
@@
 $EndComp
 $Comp
-L Device:CP1 C40
+L Device:C C40
 U 1 1 616B0985
 P 15150 4300
@@
 $EndComp
 $Comp
-L Device:CP1 C41
+L Device:C C41
 U 1 1 616EC86F
 P 15400 4300
@@
 	13300 7650 13150 7650
 $Comp
-L Device:CP1 C42
+L Device:C C42
 U 1 1 613F6646
 P 15650 4300
