File: Modules/DCDC_BuckBoost(TPS61088+MP1495S)_(Bat to 5V-3v3-2v5-1v5-1v2 3A)/PowerSupply.kicad_pcb (KiCad board)
At the start: 4 copper layers, 56 x 23.9 mm, 97 parts, among them J1 Conn_01x14, J10 Conn_01x01, J2 Conn_01x01, J3 Conn_01x01, J4 Conn_01x01, J5 Conn_01x01, J6 Conn_01x01, J7 Conn_01x01, J8 Conn_01x01, J9 Conn_01x01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

Commit message: update PowerSupply(in Kicad6)
Routing:
- net GND: track 62.1 -> 53.7 mm
- net +1V2: track 125.1 -> 122.0 mm
- net +3V3: track 219.9 -> 218.3 mm
- net Net-(2V5-Pad3): track 53.5 -> 52.6 mm
- net +5V: vias 27 -> 26
Other:
- net class Default removed
