File: Modules/DCDC_BuckBoost(TPS61088+MP2145S)_(Bat to 5V-3v3-2v5-1v5-1v2 6A)/PowerSupply.kicad_pcb (KiCad board)
At the start: 4 copper layers, 56 x 23.9 mm, 94 parts, among them J1 Conn_01x14, J10 Conn_01x01, J11 Conn_01x01, J2 Conn_01x01, J3 Conn_01x01, J4 Conn_01x01, J6 Conn_01x01, J7 Conn_01x01, J8 Conn_01x01, J9 Conn_01x01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

Commit message: update PowerSupply(in Kicad6)
Routing:
- net +5V: track 765.8 -> 265.3 mm, vias 54 -> 49
- net GND: track 45.6 -> 28.0 mm
- net +1V2: track 126.5 -> 120.0 mm
- net Net-(R19-Pad2): track 6.10 -> 2.84 mm
- net Net-(R10-Pad1): track 6.11 -> 2.91 mm
- net Net-(R21-Pad2): track 5.90 -> 2.88 mm
- net Net-(R27-Pad2): track 5.86 -> 2.96 mm
- net Net-(C21-Pad1): track 5.42 -> 4.02 mm
- net Net-(C20-Pad1): track 5.28 -> 3.91 mm
- net +1V5: track 132.7 -> 131.4 mm
- net Net-(C31-Pad1): track 5.32 -> 4.04 mm
- net Net-(C10-Pad1): track 5.40 -> 4.34 mm
- net PG_1.5: track 4.55 -> 3.54 mm
- net PG_3.3: track 4.55 -> 3.64 mm
- net PG_2.5: track 4.68 -> 3.79 mm
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- added copper zone on F.Cu, net +5V
Other:
- net class Default removed
