File: Modules/DCDC_BuckBoost(TPS61088+MP1495S)_(Bat to 5V+3V3+2V5+1V5+1V2 3A)/PowerSupply.kicad_pcb (KiCad board)
At the start: 4 copper layers, 56 x 23.9 mm, 97 parts, among them J1 Conn_01x14, J10 Conn_01x01, J2 Conn_01x01, J3 Conn_01x01, J4 Conn_01x01, J5 Conn_01x01, J6 Conn_01x01, J7 Conn_01x01, J8 Conn_01x01, J9 Conn_01x01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

Commit message: re-saved by kicad6
Parts:
- L6: value 1.8uH -> 1.5uH
Connections:
- PCI1 pad A12: (no net) -> unconnected-(PCI1-PadA12)
- PCI1 pad A13: (no net) -> unconnected-(PCI1-PadA13)
- PCI1 pad A14: (no net) -> unconnected-(PCI1-PadA14)
- PCI1 pad A15: (no net) -> unconnected-(PCI1-PadA15)
- PCI1 pad A16: (no net) -> unconnected-(PCI1-PadA16)
- PCI1 pad A17: (no net) -> unconnected-(PCI1-PadA17)
- PCI1 pad A18: (no net) -> unconnected-(PCI1-PadA18)
- U1 pad 13: (no net) -> unconnected-(U1-Pad13)
