File: Modules/DCDC_BuckBoost(TPS61088+MP1495S)_(Bat to 5V+3V3+2V5+1V5+1V2 3A)/PowerSupply.kicad_sch (KiCad schematic)
At the start: 97 parts, among them J1 Conn_01x14, J10 Conn_01x01, J2 Conn_01x01, J3 Conn_01x01, J4 Conn_01x01, J5 Conn_01x01, J6 Conn_01x01, J7 Conn_01x01, J8 Conn_01x01, J9 Conn_01x01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

Commit message: Sort Out
Parts:
- U1: footprint IC_TPS61088RHLR -> Lib:IC_TPS61088RHLR
Connections:
- net +1V2 renamed 1.2V
- net +1V5 renamed 1.5V
- net +2V5 renamed 2.5V
- net +3V3 renamed 3.3V
- net +5V renamed 5V
Other:
- moved on the sheet: 1V2, 1V5, 2V5, 3V3, C1, C10, C11, C12, C13, C14, C15, C16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
