File: Modules/DCDC_BuckBoost(TPS61088+MP2145S)_(Bat to 5V+3V3+2V5+1V5+1V2 6A)/PowerSupply.kicad_pcb (KiCad board)
At the start: 4 copper layers, 56 x 23.9 mm, 94 parts, among them J1 Conn_01x14, J10 Conn_01x01, J11 Conn_01x01, J2 Conn_01x01, J3 Conn_01x01, J4 Conn_01x01, J6 Conn_01x01, J7 Conn_01x01, J8 Conn_01x01, J9 Conn_01x01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

Commit message: re-saved by kicad6
Parts:
- removed REF**: ESD-Logo_6.6x6mm_SilkScreen, Symbol:ESD-Logo_6.6x6mm_SilkScreen
- removed REF**: Polarity_Center_Negative_6mm_SilkScreen, Symbol:Polarity_Center_Negative_6mm_SilkScreen
Connections:
- PCI1 pad A12: (no net) -> unconnected-(PCI1-PadA12)
- PCI1 pad A13: (no net) -> unconnected-(PCI1-PadA13)
- PCI1 pad A14: (no net) -> unconnected-(PCI1-PadA14)
- PCI1 pad A15: (no net) -> unconnected-(PCI1-PadA15)
- PCI1 pad A16: (no net) -> unconnected-(PCI1-PadA16)
- PCI1 pad A17: (no net) -> unconnected-(PCI1-PadA17)
- PCI1 pad A18: (no net) -> unconnected-(PCI1-PadA18)
- U1 pad 13: (no net) -> unconnected-(U1-Pad13)
