File: Modules/@Amplifier(INA848+ADA3894-2)_(60+36dB)_(10uV-1mV)/Amplifier.kicad_pcb (KiCad board)
At the start: 4 copper layers, 81.9 x 14.8 mm, 59 parts, among them J1 Conn_01x04, J2 Conn_01x01_Female, J3 Conn_01x03_Female, J4 Conn_01x02_Male, J5 Conn_01x01_Female, U1 TPS7A4901DGNR, U2 TPS7A3001DGNT, U3 ina848, U4 ADA4898-2, U5 ADA4898-2

Commit message: Sort Out
Connections:
- J1 pad 1: (no net) -> unconnected-(J1-Pad1)
- J1 pad 3: (no net) -> unconnected-(J1-Pad3)
- J1 pad 5: (no net) -> unconnected-(J1-Pad5)
- U1 pad 7: (no net) -> unconnected-(U1-Pad7)
- U2 pad 7: (no net) -> unconnected-(U2-Pad7)
