File: Modules/BatProtector(BQ2970)_(4.2V 4.5A 7A)/BatProtector_(4.2V 4.5A 7A).kicad_pcb (KiCad board)
At the start: 2 copper layers, 12.2 x 11.9 mm, 8 parts, among them U1 BQ2970, U3 CSD16406Q3, U4 CSD16406Q3

Commit message: Sort Out
Parts:
- moved U4 3.18 mm to (128.0, 77.2)
- moved U3 3.17 mm to (128.0, 80.5)
Connections:
- R7 pad 1: (no net) -> BAT+
- U1 pad 1: (no net) -> unconnected-(U1-Pad1)
Routing:
- net Net-(U3-Pad5): track 9.44 -> 14.3 mm
- net (no net): track 4.83 -> 0.00 mm
Other:
- net class Default removed
