File: Modules/LDO_BatCharger(BQ21040+BQ2970)_(USB to 4.2V 0.54A)/LDO_BatCharger(BQ21040).kicad_pcb (KiCad board)
At the start: 2 copper layers, 21.8 x 14.1 mm, 21 parts, among them J1 Conn_01x01, J2 Conn_01x01, J3 Conn_01x01, J4 Conn_01x01, J5 Conn_01x01, J6 Conn_01x01, J7 Conn_01x01, U1 BQ2970, U2 BQ21040, U3 CSD16406Q3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

Commit message: Sort Out
Connections:
- U1 pad 1: (no net) -> unconnected-(U1-Pad1)
Routing:
- net Net-(U3-Pad5): track 9.44 -> 14.3 mm
- net (no net): track 4.83 -> 0.00 mm
Other:
- net class Default removed
