File: Modules/@WirelessPowerP40_Receiver(TS61002+TS80003)/WirelessPowerP40_Receiver.kicad_pcb (KiCad board)
At the start: 4 copper layers, 53 x 53 mm, 163 parts, among them J1 Conn_01x02_Male, J2 I2C, J3 I2C, J4 I2C, J5 COIL 24uH, J6 Conn_01x02_Male, J7 Conn_01x02_Male, Q1 2N7002, Q2 2N7002, Q3 2N7002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

Commit message: Sort Out
Connections:
- H1 pad 1: (no net) -> unconnected-(H1-Pad1)
- H2 pad 1: (no net) -> unconnected-(H2-Pad1)
- H3 pad 1: (no net) -> unconnected-(H3-Pad1)
- H4 pad 1: (no net) -> unconnected-(H4-Pad1)
- U1 pad 6: (no net) -> unconnected-(U1-Pad6)
- U1 pad 7: (no net) -> unconnected-(U1-Pad7)
