File: Modules/@WirelessPowerP40_Receiver(TS61002+TS80003)/WirelessPowerP40_Receiver.kicad_sch (KiCad schematic)
At the start: 163 parts, among them J1 Conn_01x02_Male, J2 I2C, J3 I2C, J4 I2C, J5 COIL 24uH, J6 Conn_01x02_Male, J7 Conn_01x02_Male, Q1 2N7002, Q2 2N7002, Q3 2N7002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

Commit message: Sort Out
Parts:
- H1, H2, H3, H4: symbol Mechanical:MountingHole -> Connector_Generic:Conn_01x01
Connections:
- no-connect marks 15 -> 19
Changed lines of the file:
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@@
   (no_connect (at 247.65 233.68))
   (no_connect (at 247.65 236.22))
+  (no_connect (at 144.78 260.35))
+  (no_connect (at 144.78 265.43))
+  (no_connect (at 144.78 270.51))
+  (no_connect (at 144.78 275.59))
   (no_connect (at 213.36 257.81))
   (no_connect (at 213.36 260.35))
@@
     (pin "2")
   )
-  (symbol (lib_id "Mechanical:MountingHole") (at 144.78 275.59 0) (unit 1)
+  (symbol (lib_id "Connector_Generic:Conn_01x01") (at 149.86 275.59 0) (unit 1)
     (in_bom yes) (on_board yes) (fields_autoplaced)
-    (property "Reference" "H4" (id 0) (at 147.32 274.32 0)
+    (property "Reference" "H4" (id 0) (at 152.4 274.32 0)
       (effects (font (size 1.27 1.27)) (justify left))
     )
-    (property "Value" "MountingHole" (id 1) (at 147.32 276.86 0)
+    (property "Value" "MountingHole" (id 1) (at 152.4 276.86 0)
       (effects (font (size 1.27 1.27)) (justify left))
     )
-    (property "Footprint" "MountingHole:MountingHole_2.2mm_M2_Pad_Via" (id 2) (at 144.78 275.59 0)
+    (property "Footprint" "MountingHole:MountingHole_2.2mm_M2_Pad_Via" (id 2) (at 149.86 275.59 0)
       (effects (font (size 1.27 1.27)) hide)
     )
-    (property "Datasheet" "~" (id 3) (at 144.78 275.59 0)
+    (property "Datasheet" "~" (id 3) (at 149.86 275.59 0)
       (effects (font (size 1.27 1.27)) hide)
     )
+    (pin "1")
   )
   (symbol (lib_id "Device:C") (at 422.91 59.69 180) (unit 1)
@@
     (pin "2")
   )
-  (symbol (lib_id "Mechanical:MountingHole") (at 144.78 265.43 0) (unit 1)
+  (symbol (lib_id "Connector_Generic:Conn_01x01") (at 149.86 265.43 0) (unit 1)
     (in_bom yes) (on_board yes) (fields_autoplaced)
-    (property "Reference" "H2" (id 0) (at 147.32 264.16 0)
+    (property "Reference" "H2" (id 0) (at 152.4 264.16 0)
       (effects (font (size 1.27 1.27)) (justify left))
     )
-    (property "Value" "MountingHole" (id 1) (at 147.32 266.7 0)
+    (property "Value" "MountingHole" (id 1) (at 152.4 266.7 0)
       (effects (font (size 1.27 1.27)) (justify left))
     )
-    (property "Footprint" "MountingHole:MountingHole_2.2mm_M2_Pad_Via" (id 2) (at 144.78 265.43 0)
+    (property "Footprint" "MountingHole:MountingHole_2.2mm_M2_Pad_Via" (id 2) (at 149.86 265.43 0)
       (effects (font (size 1.27 1.27)) hide)
     )
-    (property "Datasheet" "~" (id 3) (at 144.78 265.43 0)
+    (property "Datasheet" "~" (id 3) (at 149.86 265.43 0)
       (effects (font (size 1.27 1.27)) hide)
     )
+    (pin "1")
   )
   (symbol (lib_id "Device:R") (at 96.52 43.18 90) (unit 1)
@@
     (pin "9")
   )
-  (symbol (lib_id "Mechanical:MountingHole") (at 144.78 260.35 0) (unit 1)
+  (symbol (lib_id "Connector_Generic:Conn_01x01") (at 149.86 260.35 0) (unit 1)
     (in_bom yes) (on_board yes)
-    (property "Reference" "H1" (id 0) (at 147.32 259.08 0)
+    (property "Reference" "H1" (id 0) (at 152.4 259.08 0)
       (effects (font (size 1.27 1.27)) (justify left))
     )
-    (property "Value" "MountingHole" (id 1) (at 147.32 261.62 0)
+    (property "Value" "MountingHole" (id 1) (at 152.4 261.62 0)
       (effects (font (size 1.27 1.27)) (justify left))
     )
-    (property "Footprint" "MountingHole:MountingHole_2.2mm_M2_Pad_Via" (id 2) (at 144.78 260.35 0)
+    (property "Footprint" "MountingHole:MountingHole_2.2mm_M2_Pad_Via" (id 2) (at 149.86 260.35 0)
       (effects (font (size 1.27 1.27)) hide)
     )
-    (property "Datasheet" "~" (id 3) (at 144.78 260.35 0)
+    (property "Datasheet" "~" (id 3) (at 149.86 260.35 0)
       (effects (font (size 1.27 1.27)) hide)
     )
+    (pin "1")
   )
   (symbol (lib_id "power:GND") (at 87.63 214.63 0) (unit 1)
@@
     (pin "2")
   )
-  (symbol (lib_id "Mechanical:MountingHole") (at 144.78 270.51 0) (unit 1)
+  (symbol (lib_id "Connector_Generic:Conn_01x01") (at 149.86 270.51 0) (unit 1)
     (in_bom yes) (on_board yes) (fields_autoplaced)
-    (property "Reference" "H3" (id 0) (at 147.32 269.24 0)
+    (property "Reference" "H3" (id 0) (at 152.4 269.24 0)
       (effects (font (size 1.27 1.27)) (justify left))
     )
-    (property "Value" "MountingHole" (id 1) (at 147.32 271.78 0)
+    (property "Value" "MountingHole" (id 1) (at 152.4 271.78 0)
       (effects (font (size 1.27 1.27)) (justify left))
     )
-    (property "Footprint" "MountingHole:MountingHole_2.2mm_M2_Pad_Via" (id 2) (at 144.78 270.51 0)
+    (property "Footprint" "MountingHole:MountingHole_2.2mm_M2_Pad_Via" (id 2) (at 149.86 270.51 0)
       (effects (font (size 1.27 1.27)) hide)
     )
-    (property "Datasheet" "~" (id 3) (at 144.78 270.51 0)
+    (property "Datasheet" "~" (id 3) (at 149.86 270.51 0)
       (effects (font (size 1.27 1.27)) hide)
     )
+    (pin "1")
   )
   (symbol (lib_id "Diode:BAS21") (at 388.62 64.77 270) (unit 1)
@@
     (pin "4")
     (pin "5")
+    (pin "6")
+    (pin "7")
     (pin "8")
     (pin "9")
