File: Modules/@WirelessPowerP40_Transmitter(TS61002+TS80003)/WirelessPowerP40_Transmitter.kicad_pcb (KiCad board)
At the start: 4 copper layers, 53 x 53 mm, 136 parts, among them J1 USBA, J2 I2C, J3 I2C, J4 Coil Therm, J5 COIL 20uH, J6 Conn_01x02_Male, J7 Conn_01x02_Male, U1 TS30041, U10 HUSB238, U2 TS94033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

Commit message: Sort Out
Connections:
- H1 pad 1: (no net) -> unconnected-(H1-Pad1)
- H2 pad 1: (no net) -> unconnected-(H2-Pad1)
- H3 pad 1: (no net) -> unconnected-(H3-Pad1)
- H4 pad 1: (no net) -> unconnected-(H4-Pad1)
- U1 pad 6: (no net) -> unconnected-(U1-Pad6)
- U1 pad 7: (no net) -> unconnected-(U1-Pad7)
