File: Modules/@WirelessPowerP40_Transmitter(TS61002+TS80003)/WirelessPowerP40_Transmitter.kicad_sch (KiCad schematic)
At the start: 136 parts, among them J1 USBA, J2 I2C, J3 I2C, J4 Coil Therm, J5 COIL 20uH, J6 Conn_01x02_Male, J7 Conn_01x02_Male, U1 TS30041, U10 HUSB238, U2 TS94033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

Commit message: Sort Out
Parts:
- H1, H2, H3, H4: symbol Mechanical:MountingHole -> Connector_Generic:Conn_01x01
- U3: symbol 74xGxx:74LVC1G66-full -> 74LVC1G66:74LVC1G66-full
Connections:
- no-connect marks 20 -> 24
Changed lines of the file:
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@@
   (junction (at 73.66 41.91) (diameter 0) (color 0 0 0 0)
   )
+  (no_connect (at 379.73 34.29))
+  (no_connect (at 379.73 29.21))
+  (no_connect (at 379.73 24.13))
+  (no_connect (at 379.73 19.05))
   (no_connect (at 165.1 36.83))
   (no_connect (at 165.1 48.26))
@@
     (pin "1")
   )
-  (symbol (lib_id "Mechanical:MountingHole") (at 391.16 30.48 0) (unit 1)
+  (symbol (lib_id "Connector_Generic:Conn_01x01") (at 384.81 34.29 0) (unit 1)
     (in_bom yes) (on_board yes) (fields_autoplaced)
-    (property "Reference" "H4" (id 0) (at 393.7 29.21 0)
+    (property "Reference" "H4" (id 0) (at 387.35 33.02 0)
       (effects (font (size 1.27 1.27)) (justify left))
     )
-    (property "Value" "MountingHole" (id 1) (at 393.7 31.75 0)
+    (property "Value" "MountingHole" (id 1) (at 387.35 35.56 0)
       (effects (font (size 1.27 1.27)) (justify left))
     )
-    (property "Footprint" "MountingHole:MountingHole_2.2mm_M2_Pad_Via" (id 2) (at 391.16 30.48 0)
+    (property "Footprint" "MountingHole:MountingHole_2.2mm_M2_Pad_Via" (id 2) (at 384.81 34.29 0)
       (effects (font (size 1.27 1.27)) hide)
     )
-    (property "Datasheet" "~" (id 3) (at 391.16 30.48 0)
+    (property "Datasheet" "~" (id 3) (at 384.81 34.29 0)
       (effects (font (size 1.27 1.27)) hide)
     )
+    (pin "1")
   )
-  (symbol (lib_id "Mechanical:MountingHole") (at 391.16 20.32 0) (unit 1)
+  (symbol (lib_id "Connector_Generic:Conn_01x01") (at 384.81 24.13 0) (unit 1)
     (in_bom yes) (on_board yes) (fields_autoplaced)
-    (property "Reference" "H2" (id 0) (at 393.7 19.05 0)
+    (property "Reference" "H2" (id 0) (at 387.35 22.86 0)
       (effects (font (size 1.27 1.27)) (justify left))
     )
-    (property "Value" "MountingHole" (id 1) (at 393.7 21.59 0)
+    (property "Value" "MountingHole" (id 1) (at 387.35 25.4 0)
       (effects (font (size 1.27 1.27)) (justify left))
     )
-    (property "Footprint" "MountingHole:MountingHole_2.2mm_M2_Pad_Via" (id 2) (at 391.16 20.32 0)
+    (property "Footprint" "MountingHole:MountingHole_2.2mm_M2_Pad_Via" (id 2) (at 384.81 24.13 0)
       (effects (font (size 1.27 1.27)) hide)
     )
-    (property "Datasheet" "~" (id 3) (at 391.16 20.32 0)
+    (property "Datasheet" "~" (id 3) (at 384.81 24.13 0)
       (effects (font (size 1.27 1.27)) hide)
     )
+    (pin "1")
   )
   (symbol (lib_id "power:GND") (at 91.44 166.37 0) (unit 1)
@@
     (pin "1")
   )
-  (symbol (lib_id "Mechanical:MountingHole") (at 391.16 15.24 0) (unit 1)
+  (symbol (lib_id "Connector_Generic:Conn_01x01") (at 384.81 19.05 0) (unit 1)
     (in_bom yes) (on_board yes)
-    (property "Reference" "H1" (id 0) (at 393.7 13.97 0)
+    (property "Reference" "H1" (id 0) (at 387.35 17.78 0)
       (effects (font (size 1.27 1.27)) (justify left))
     )
-    (property "Value" "MountingHole" (id 1) (at 393.7 16.51 0)
+    (property "Value" "MountingHole" (id 1) (at 387.35 20.32 0)
       (effects (font (size 1.27 1.27)) (justify left))
     )
-    (property "Footprint" "MountingHole:MountingHole_2.2mm_M2_Pad_Via" (id 2) (at 391.16 15.24 0)
+    (property "Footprint" "MountingHole:MountingHole_2.2mm_M2_Pad_Via" (id 2) (at 384.81 19.05 0)
       (effects (font (size 1.27 1.27)) hide)
     )
-    (property "Datasheet" "~" (id 3) (at 391.16 15.24 0)
+    (property "Datasheet" "~" (id 3) (at 384.81 19.05 0)
       (effects (font (size 1.27 1.27)) hide)
     )
+    (pin "1")
   )
   (symbol (lib_id "power:GND") (at 204.47 134.62 0) (unit 1)
@@
     (pin "S4")
   )
-  (symbol (lib_id "Mechanical:MountingHole") (at 391.16 25.4 0) (unit 1)
+  (symbol (lib_id "Connector_Generic:Conn_01x01") (at 384.81 29.21 0) (unit 1)
     (in_bom yes) (on_board yes) (fields_autoplaced)
-    (property "Reference" "H3" (id 0) (at 393.7 24.13 0)
+    (property "Reference" "H3" (id 0) (at 387.35 27.94 0)
       (effects (font (size 1.27 1.27)) (justify left))
     )
-    (property "Value" "MountingHole" (id 1) (at 393.7 26.67 0)
+    (property "Value" "MountingHole" (id 1) (at 387.35 30.48 0)
       (effects (font (size 1.27 1.27)) (justify left))
     )
-    (property "Footprint" "MountingHole:MountingHole_2.2mm_M2_Pad_Via" (id 2) (at 391.16 25.4 0)
+    (property "Footprint" "MountingHole:MountingHole_2.2mm_M2_Pad_Via" (id 2) (at 384.81 29.21 0)
       (effects (font (size 1.27 1.27)) hide)
     )
-    (property "Datasheet" "~" (id 3) (at 391.16 25.4 0)
+    (property "Datasheet" "~" (id 3) (at 384.81 29.21 0)
       (effects (font (size 1.27 1.27)) hide)
     )
+    (pin "1")
   )
   (symbol (lib_id "Device:R") (at 270.51 49.53 90) (unit 1)
@@
       (effects (font (size 1.27 1.27)) (justify left))
     )
-    (property "Value" "1uF 50V" (id 1) (at 40.64 87.63 0)
+    (property "Value" "1uF 50V" (id 1) (at 40.64 88.9 0)
       (effects (font (size 1.27 1.27)) (justify left))
     )
@@
     (pin "2")
   )
-  (symbol (lib_id "74xGxx:74LVC1G66-full") (at 115.57 214.63 0) (unit 1)
+  (symbol (lib_id "74LVC1G66:74LVC1G66-full") (at 115.57 214.63 0) (unit 1)
     (in_bom yes) (on_board yes)
     (property "Reference" "U3" (id 0) (at 120.65 208.28 0))
@@
     (pin "4")
     (pin "5")
+    (pin "6")
+    (pin "7")
     (pin "8")
     (pin "9")

Commit message: Sort Out
Parts:
- U10: symbol Hynetek:HUSB238 -> HUSB238:HUSB238
Changed lines of the file:
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@@
     (pin "2")
   )
-  (symbol (lib_id "Hynetek:HUSB238") (at 156.21 44.45 0) (unit 1)
+  (symbol (lib_id "HUSB238:HUSB238") (at 156.21 44.45 0) (unit 1)
     (in_bom yes) (on_board yes) (fields_autoplaced)
     (property "Reference" "U10" (id 0) (at 156.21 30.3743 0))
