File: Modules/WirelessPowerReceiver(BQ51013+BQ24040+BQ2970)_(5V 1A)/WirelessPower.kicad_sch (KiCad schematic)
At the start: 46 parts, among them J1 Conn_01x01_Female, J2 Conn_01x01_Female, J3 Conn_01x01_Female, J4 Conn_01x01_Female, J5 BAT, J6 AC, J7 Conn_01x14, U1 BQ2971, U2 BQ51013BRHLR, U3 CSD16406Q3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

Commit message: Sort Out
Parts:
- J1, J2, J3, J4: symbol Connector:Conn_01x01_Female -> Mechanical:MountingHole
- U1: symbol BC:BQ2971 -> BQ297X:BQ297X
- U2: footprint IC_MSP430FR2522IRHLR -> lib:BQ51013BRHLR
- U3, U4: footprint BC:CSD16406Q3 -> lib:CSD16406Q3; symbol BC:CSD16406Q3 -> CSD16406Q3:CSD16406Q3
- U5: footprint SON40P200X200X80-11N -> lib:BQ24040DSQT
Connections:
- no-connect marks 6 -> 2
