File: Modules/#USB2_Jtag_Bridge_(FT232HQ)/USB2_Jtag_Bridge.kicad_sch (KiCad schematic)
At the start: 1 part

Commit message: Update USB2_Jtag_Bridge
Parts:
- added C1, C10, C12, C14, C15, C2, C5, C7, C9: 0.1uF, Capacitor_SMD:C_0402_1005Metric, symbol Device:C
- added C11, C13, C16, C17, C6, C8: 10uF, Capacitor_SMD:C_0402_1005Metric, symbol Device:C
- added C3, C4: 27pF, Capacitor_SMD:C_0402_1005Metric, symbol Device:C
- added D1: LED, LED_SMD:LED_0402_1005Metric, symbol Device:LED
- added J1: USB-C16PSMT01, Connector_USB:USB_C_Receptacle_XKB_U262-16XN-4BVC11, symbol USB-C16PSMT01:CQ-USB-C16PSMT01
- added J2: Conn_01x06_Male, Connector_PinHeader_2.54mm:PinHeader_1x06_P2.54mm_Vertical, symbol Connector:Conn_01x06_Male
- added L1: 4.7uF, Inductor_SMD:L_Taiyo-Yuden_NR-30xx, symbol Device:L
- added R10: 1M, Resistor_SMD:R_0402_1005Metric, symbol Device:R
- added R11: 20R, Resistor_SMD:R_0402_1005Metric, symbol Device:R
- added R12: 51K, Resistor_SMD:R_0402_1005Metric, symbol Device:R
- added R13: 13K, Resistor_SMD:R_0402_1005Metric, symbol Device:R
- added R14: 41.2K, Resistor_SMD:R_0402_1005Metric, symbol Device:R
- added R3: 12K, Resistor_SMD:R_0402_1005Metric, symbol Device:R
- added R4, R5, R6, R7: 10K, Resistor_SMD:R_0402_1005Metric, symbol Device:R
- added R8: 2K, Resistor_SMD:R_0402_1005Metric, symbol Device:R
- added R9: 3K, Resistor_SMD:R_0402_1005Metric, symbol Device:R
- added U2: 93LC56BxxOT, Package_TO_SOT_SMD:SOT-23-6, symbol Memory_EEPROM:93LCxxBxxOT
- added U3: mp9442, Package_TO_SOT_SMD:TSOT-23-8, symbol MP9442:mp9442
- added Y1: 12M, Crystal:Crystal_SMD_TXC_9HT11-2Pin_2.0x1.2mm_HandSoldering, symbol Device:Crystal
- U1: renamed from U?; footprint (none) -> Package_DFN_QFN:QFN-48-1EP_8x8mm_P0.5mm_EP6.2x6.2mm
Connections:
- net at U1.1 (XCSI): now also C3.2, Y1.1
- net VSS: now reaches U1.10 (GND)
- net VSS: now also U1.11 (GND), U1.22 (GND), U1.23 (GND), U1.35 (GND), U1.36 (GND), U1.4 (AGND), U1.41 (AGND), U1.42 (TEST), U1.47 (GND), U1.48 (GND), U1.49 (EP), U1.9 (AGND), C1.2, C10.2, C11.2, C12.2, C13.2, C14.2, C16.2, C17.2, C2.2, C3.1, C4.1, C5.2, C6.2, C7.2, C8.2, C9.2, D1.1 (K), J1.A1 (GND), J1.A12 (GND), J1.B1 (GND), J1.B12 (GND), J1.S1 (SHIELD), J2.5 (Pin_5), R13.1, R3.2, U2.2 (GND), U3.4 (GND)
- net +3V3: now reaches U1.12 (VCCIO)
- net +3V3: now also U1.24 (VCCIO), U1.3 (VPHY), U1.39 (VCCD), U1.46 (VCCIO), U1.8 (VPLL), C10.1, C6.1, C7.1, C8.1, C9.1, R4.2, R5.1, R6.1, R7.1, U2.6 (VCC)
- net TCK: now reaches U1.13 (ADBUS0)
- net TCK: now also J2.1 (Pin_1)
- net TDI: now reaches U1.14 (ADBUS1)
- net TDI: now also J2.2 (Pin_2)
- net TDO: now reaches U1.15 (ADBUS2)
- net TDO: now also J2.3 (Pin_3)
- net TMS: now reaches U1.16 (ADBUS3)
- net TMS: now also J2.4 (Pin_4)
- net at U1.2 (XCSO): now also C4.2, Y1.2
- net RESET: now reaches U1.34 (~{RESET})
- net RESET: now also C5.1, R4.1
- net at U1.37 (VCCA): now also C2.1
- net at U1.38 (VCCCORE): now also C1.1
- net VBUS: now reaches U1.40 (VREGIN)
- net VBUS: now also C11.1, C12.1, C13.1, J1.A4 (VBUS), J1.A9 (VBUS), J1.B4 (VBUS), J1.B9 (VBUS), R10.2, R9.2, U3.2 (IN)
- net EEP_D: now reaches U1.43 (EEDATA)
- net EEP_D: now also R8.2, U2.3 (DI)
- net EEP_CLK: now reaches U1.44 (EECLK)
- net EEP_CLK: now also R7.2, U2.4 (CLK)
- net EEP_CS: now reaches U1.45 (EECS)
- net EEP_CS: now also R5.2, U2.5 (CS)
- net at U1.5 (REF): now also R3.1
- net DM: now reaches U1.6 (DM)
- net DM: now also J1.A7 (DN1), J1.B7 (DN2)
- net DP: now reaches U1.7 (DP)
- net DP: now also J1.A6 (DP1), J1.B6 (DP2)
- new net: R6.2, R8.1, U2.1 (DO)
- new net: R12.1, R13.2, R14.2
- new net: C15.1, R11.1
- new net: R11.2, U3.5 (BST)
- new net: C15.2, L1.1, U3.3 (SW)
- new net: D1.2 (A), R9.1, U3.1 (PG)
- new net: R10.1, U3.6 (EN)
- new net: C14.1, U3.7 (VCC)
- new net: R12.2, U3.8 (FB)
- new net 3.3V: C16.1, C17.1, J2.6 (Pin_6), L1.2, R14.1
- no-connect marks 0 -> 18
