File: Projects/USB3G2_SATA3_Bridge(JMS580)/USB3G2_SATA3_Bridge(JMS580).kicad_pcb (KiCad board)
At the start: 4 copper layers, 40.4 x 31.1 mm, 75 parts, among them J1 ATA-A, J2 USB_C_Receptacle, Q1 MMBT3904LT1G(1AM), Q2 AO3401A, Q3 AO3400A, U1 W25Q32JVZP, U2 JMS580, U3 FP6381A, Y1 Crystal_GND24

Commit message: Fix layout
Parts:
- R10: value 0R -> 0R / NS
Routing:
- net VBUS: track 41.9 -> 37.2 mm, vias 16 -> 15
- net GND: vias 120 -> 119

Commit message: Sort Out
Parts:
- L1: value 4R7 -> 4R7 / NS
Changed lines of the file:
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@@
       (effects (font (size 0.6 0.6) (thickness 0.1)))
     )
-    (fp_text value "4R7" (at -0.1 2.8) (layer "F.Fab")
+    (fp_text value "4R7 / NS" (at -0.1 2.8) (layer "F.Fab")
       (effects (font (size 1 1) (thickness 0.15)))
     )

Commit message: Sort Out
Parts:
- H4: value MountingHole -> Symbol
Connections:
- net 3V3 renamed LDO_33
- H1 pad 1: (no net) -> unconnected-(H1-Pad1)
- H2 pad 1: (no net) -> unconnected-(H2-Pad1)
- H3 pad 1: (no net) -> unconnected-(H3-Pad1)

Commit message: Remove PCBsch useless layers
Changed lines of the file:
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@@
     (38 "B.Mask" user)
     (39 "F.Mask" user)
-    (40 "Dwgs.User" user "User.Drawings")
-    (41 "Cmts.User" user "User.Comments")
-    (42 "Eco1.User" user "User.Eco1")
-    (43 "Eco2.User" user "User.Eco2")
     (44 "Edge.Cuts" user)
     (45 "Margin" user)
     (46 "B.CrtYd" user "B.Courtyard")
     (47 "F.CrtYd" user "F.Courtyard")
-    (48 "B.Fab" user)
-    (49 "F.Fab" user)
-    (50 "User.1" user)
-    (51 "User.2" user)
-    (52 "User.3" user)
-    (53 "User.4" user)
-    (54 "User.5" user)
-    (55 "User.6" user)
-    (56 "User.7" user)
-    (57 "User.8" user)
-    (58 "User.9" user)
   )
   (setup
@@
   (gr_line locked (start 113.54 67.98) (end 114.11 67.98) (layer "Edge.Cuts") (width 0.1))
   (gr_line locked (start 153.010876 69.99) (end 152.475 69.99) (layer "Edge.Cuts") (width 0.1))
-  (gr_arc locked (start 150.407684 62.649597) (mid 152.597143 63.558176) (end 153.5 65.75) (layer "Edge.Cuts") (width 0.1))
+  (gr_arc locked (start 150.407684 62.649597) (mid 152.597142 63.558176) (end 153.5 65.75) (layer "Edge.Cuts") (width 0.1))
   (gr_arc locked (start 113.1 65.75) (mid 114.008087 63.557684) (end 116.200403 62.649597) (layer "Edge.Cuts") (width 0.1))
   (gr_line locked (start 113.1 67.48) (end 113.1 65.75) (layer "Edge.Cuts") (width 0.1))
