File: Projects/#FPGA_XC6SLX25(FTG256)_CoreBoard/XC6SLX25(FTG256)_CoreBoard.kicad_pcb (KiCad board)
At the start: 6 copper layers, 69.6 x 30 mm, 148 parts, among them J1 MTA18ASF2G72HZ-2G3A1, U1 XC6SLX25-FTG256, U2 W25Q128JVS, U3 TPS51200DRC, U4 MP214x, U5 MP214x, U6 MP214x, U7 MP214x, X1 ECS-2520MV-xxx-xx

Commit message: Update XC6SLX25(FTG256)_CoreBoard
Parts:
- moved RN6 22.5 mm to (119.9, 74.9), turned to -90 degrees
- moved RN4 22.1 mm to (112.4, 74.9), turned to -90 degrees
- moved RN2 21.6 mm to (114.9, 74.9), turned to -90 degrees
- moved RN1 21.1 mm to (117.4, 74.9), turned to -90 degrees
- moved RN3 17.5 mm to (108.5, 77.7), turned to 0 degrees
- moved RN5 14.4 mm to (108.5, 80.2), turned to 180 degrees
- moved C49 0.36 mm to (121.2, 84.5)
- moved C46 0.30 mm to (121.2, 77.3)
- moved C47 0.30 mm to (121.2, 79.9)
- moved C48 0.30 mm to (121.2, 81.7)
- moved C50 0.30 mm to (121.2, 86.9)
- moved C51 0.30 mm to (121.2, 89.5)
- moved C52 0.30 mm to (111.1, 87.5)
- moved C53 0.30 mm to (111.1, 85.7)
- moved C54 0.30 mm to (111.1, 82.9)
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Connections:
- RN7 pad 5: /DDR_D1 -> /DDR_D2
- RN7 pad 7: /DDR_D2 -> /DDR_D1
- RN8 pad 5: /DDR_D7 -> /DDR_D5
- RN8 pad 6: /DDR_D6 -> /DDR_D7
- RN8 pad 7: /DDR_D5 -> /DDR_D4
- RN8 pad 8: /DDR_D4 -> /DDR_D6
- RN9 pad 7: /DDR_D9 -> /DDR_D11
- RN9 pad 8: /DDR_D11 -> /DDR_D9
Routing:
- net /DDR_CLK+: track 2.58 -> 18.1 mm
- net /DDR_CLK-: track 2.33 -> 17.8 mm
- net /DDR_D5: track 1.16 -> 14.6 mm
- net /DDR_D7: track 1.16 -> 13.7 mm
- net +1V5: track 39.6 -> 51.3 mm
- net /DDR_LDQS-: track 0.59 -> 12.0 mm
- net /DDR_LDQS+: track 0.59 -> 12.0 mm
- net /DDR_D4: track 1.55 -> 10.6 mm
- net /DDR_D6: track 1.55 -> 9.56 mm
- net +2V5: track 9.26 -> 17.1 mm
- net +1V2: track 31.4 -> 39.2 mm
- net +3V3: track 17.7 -> 25.6 mm
- net /DDR_UDM: track 10.8 -> 8.85 mm
- net /DDR_D9: track 9.21 -> 10.9 mm
- net /DDR_D0: track 10.6 -> 9.10 mm
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