File: Projects/#FPGA_XC6SLX25(FTG256)_CoreBoard_Ep_OnlyIO/XC6SLX25(FTG256)_BaseBoard_OnlyIO.kicad_pcb (KiCad board)
At the start: 6 copper layers, 1 part, among them J1 2309411-1

Commit message: update FPGA_XC6SLX25_BaseBoard_OnlyIO
Parts:
- added J2: Conn_01x30, Connector_PinSocket_2.54mm:PinSocket_1x30_P2.54mm_Vertical, F.Cu at (109.7, 122.9)
- added J3: Conn_01x30, Connector_PinSocket_2.54mm:PinSocket_1x30_P2.54mm_Vertical, F.Cu at (109.7, 138.0)
- added J4: Conn_01x30, Connector_PinSocket_2.54mm:PinSocket_1x30_P2.54mm_Vertical, F.Cu at (109.7, 127.9)
- added J5: Conn_01x30, Connector_PinSocket_2.54mm:PinSocket_1x30_P2.54mm_Vertical, F.Cu at (109.7, 133.0)
