File: Module/#ESP32_S2_WROVER_EVB/ESP32_S2_WROVER_EVB.kicad_sch (KiCad schematic)
At the start: 90 parts, among them J1 CQ-USB-C16PSMT01, J3 Motor, J4 ADC_IN1, J5 ADC_IN2, J6 ADC_REF, Q1 Q_NPN_BEC, Q2 Q_NPN_BEC, SW1 SW_Push, SW2 SW_Push, U1 ESP32_S2_WROVER, U2 MP214x, U3 CP2102N-QFN28, U4 SN74LV1T34DBV, U5 GC9A01_CST916D_240*240, U8 VEML7700

Commit message: update ESP-S2-Wrover module
Parts:
- added C28: (no value), symbol Device:C
- added H1, H2, H3, H4, H5, H6: (no value), symbol Mechanical:MountingHole_Pad
- added J7, J8: (no value), symbol Connector_Generic_MountingPin:Conn_01x08_MountingPin
- C1, C2: value 10uF -> (none); footprint Capacitor_SMD:C_0603_1608Metric -> (none)
- C10, C16, C18, C19, C20, C21, C22, C23, C24, C25, C26, C27, C4, C5, C9: value 0.1uF -> (none); footprint Capacitor_SMD:C_0402_1005Metric -> (none)
- C11, C13: value 22uF -> (none); footprint Capacitor_SMD:C_0603_1608Metric -> (none)
- C12, C3, C6, C7, C8: value 1uF -> (none); footprint Capacitor_SMD:C_0402_1005Metric -> (none)
- C14, C15, C17: value 10uF -> (none); footprint Capacitor_SMD:C_0402_1005Metric -> (none)
- D1, D2, D3, D4, D5: value LED -> (none); footprint LED_SMD:LED_0402_1005Metric -> (none)
- D10, D11, D12, D13, D6, D7, D8, D9: value SK6812 -> (none); footprint LED_SMD:LED_SK6812_PLCC4_5.0x5.0mm_P3.2mm -> (none); symbol LED:SK6812 -> SK6812:SK6812-4020
- J1: value CQ-USB-C16PSMT01 -> (none); footprint Connector_USB:USB_C_Receptacle_XKB_U262-16XN-4BVC11 -> (none)
- J2: footprint lib:microSD -> (none)
- J3: value Motor -> (none); footprint Connector_JST:JST_PH_S3B-PH-SM4-TB_1x03-1MP_P2.00mm_Horizontal -> (none)
- J4: value ADC_IN1 -> (none); footprint Connector_JST:JST_ACH_BM02B-ACHSS-GAN-ETF_1x02-1MP_P1.20mm_Vertical -> (none)
- J5: value ADC_IN2 -> (none); footprint Connector_JST:JST_ACH_BM02B-ACHSS-GAN-ETF_1x02-1MP_P1.20mm_Vertical -> (none)
- J6: value ADC_REF -> (none); footprint Connector_JST:JST_ACH_BM02B-ACHSS-GAN-ETF_1x02-1MP_P1.20mm_Vertical -> (none)
- L1: value 0.47uH -> (none); footprint Inductor_SMD:L_Taiyo-Yuden_NR-40xx -> (none)
- Q1, Q2: value Q_NPN_BEC -> (none); footprint Package_TO_SOT_SMD:SOT-23 -> (none)
- R1, R17, R18, R25, R26, R27, R9: value 10K -> (none); footprint Resistor_SMD:R_0402_1005Metric -> (none)
- R10: value 200K -> (none); footprint Resistor_SMD:R_0402_1005Metric -> (none)
- R11: value 44.2K -> (none); footprint Resistor_SMD:R_0402_1005Metric -> (none)
- R12, R4: value 470R -> (none); footprint Resistor_SMD:R_0402_1005Metric -> (none)
- R13: value 1K -> (none); footprint Resistor_SMD:R_0402_1005Metric -> (none)
- R14, R15, R19, R20, R21, R8: value 4K7 -> (none); footprint Resistor_SMD:R_0402_1005Metric -> (none)
- R16, R2, R3, R6: value 2K -> (none); footprint Resistor_SMD:R_0402_1005Metric -> (none)
- R22: value 8R -> (none); footprint Resistor_SMD:R_0805_2012Metric -> (none)
- R23, R24: value 1.5K -> (none); footprint Resistor_SMD:R_0402_1005Metric -> (none)
- R5, R7: value 100K -> (none); footprint Resistor_SMD:R_0402_1005Metric -> (none)
- RN1: value 10K -> (none); footprint Resistor_SMD:R_Array_Convex_8x0602 -> (none)
- SW1, SW2: value SW_Push -> (none); footprint Button_Switch_SMD:SW_Push_1P1T_NO_Vertical_Wuerth_434133025816 -> (none)
- U1: value ESP32_S2_WROVER -> (none); footprint lib:ESP32-WROVER -> (none)
- U2: value MP214x -> (none); footprint lib:MP2145 -> (none)
- U3: value CP2102N-QFN28 -> (none); footprint Package_DFN_QFN:QFN-28-1EP_5x5mm_P0.5mm_EP3.35x3.35mm -> (none)
- U4: value SN74LV1T34DBV -> (none); footprint Package_TO_SOT_SMD:SOT-23-5 -> (none)
- U5: value GC9A01_CST916D_240*240 -> (none); footprint Connector_FFC-FPC:Hirose_FH12-15S-0.5SH_1x15-1MP_P0.50mm_Horizontal -> (none); symbol LCD:GC9A01_CST916D_240*240 -> LCD:GC9A01_CST816D_240*240
- U7: footprint Package_SO:SOIC-8_3.9x4.9mm_P1.27mm -> (none)
- U8: value VEML7700 -> (none); footprint lib:VEML7700 -> (none)
Connections:
- net +3V3: now also R27.1, J7.4 (Pin_4); no longer C14.1, C16.1, R27.2, U5.10 (TP_VDD), U5.3 (BL_A), U5.4 (DP_VDD)
- net +5V: now also D10.2 (VDD), D11.2 (VDD), D12.2 (VDD), D13.2 (VDD), D6.2 (VDD), D7.2 (VDD), D8.2 (VDD), D9.2 (VDD), C28.1; no longer D10.3 (VDD), D11.3 (VDD), D12.3 (VDD), D13.3 (VDD), D6.3 (VDD), D7.3 (VDD), D8.3 (VDD), D9.3 (VDD)
- net DP_CS: now also R27.2, J7.7 (Pin_7); no longer R27.1, U5.6 (DP_CS)
- net ESP_I2C_SCL: now also J7.2 (Pin_2); no longer U5.14 (TP_SDA)
- net ESP_I2C_SDA: now also J7.1 (Pin_1); no longer U5.15 (TP_SCL)
- net ESP_SPI_CLK: now also J7.6 (Pin_6); no longer U5.7 (DP_CLK)
- net ESP_SPI_MISO: now also J7.8 (Pin_8); no longer U5.5 (DP_DC)
- net ESP_SPI_MOSI: now also J7.5 (Pin_5); no longer U5.8 (DP_SDA)
- net GND: now also D10.4 (VSS), D11.4 (VSS), D12.4 (VSS), D13.4 (VSS), D6.4 (VSS), D7.4 (VSS), D8.4 (VSS), D9.4 (VSS), C28.2, J7.3 (Pin_3), J7.MP (MountPin); no longer C14.2, C16.2, D10.1 (VSS), D11.1 (VSS), D12.1 (VSS), D13.1 (VSS), D6.1 (VSS), D7.1 (VSS), D8.1 (VSS), D9.1 (VSS), R22.1, U5.1 (GND), U5.11 (GND), U5.MP
- net TMC_UH: now also RN1.8 (R8.1); no longer RN1.1 (R1.1)
- net TMC_UL: now also RN1.5 (R5.1); no longer RN1.2 (R2.1)
- net TMC_VH: now also RN1.7 (R7.1); no longer RN1.3 (R3.1)
- net TMC_VL: now also RN1.1 (R1.1); no longer RN1.4 (R4.1)
- net TMC_WH: now also RN1.6 (R6.1); no longer RN1.5 (R5.1)
- net TMC_WL: now also RN1.4 (R4.1); no longer RN1.6 (R6.1)
- net at U4.4 (Y): now also D6.1 (DIN); no longer D6.2 (DIN)
- new net: D6.3 (DOUT), D7.1 (DIN)
- new net: D7.3 (DOUT), D8.1 (DIN)
- new net: D11.3 (DOUT), D12.1 (DIN)
- new net: D12.3 (DOUT), D13.1 (DIN)
- new net: D8.3 (DOUT), D9.1 (DIN)
- new net: D10.1 (DIN), D9.3 (DOUT)
- new net: D10.3 (DOUT), D11.1 (DIN)
- new net Screen_DP_CLK: J8.6 (Pin_6), U5.7 (DP_CLK)
- new net Screen_DP_CMD: J8.8 (Pin_8), U5.5 (DP_DC)
- new net Screen_DP_CS: J8.7 (Pin_7), U5.6 (DP_CS)
- new net Screen_DP_DATA: J8.5 (Pin_5), U5.8 (DP_SDA)
- new net Screen_GND: C14.2, C16.2, J8.3 (Pin_3), J8.MP (MountPin), R22.1, U5.1 (GND), U5.11 (GND), U5.MP
- new net Screen_TP_SCL: J8.2 (Pin_2), U5.14 (TP_SDA)
- new net Screen_TP_SDA: J8.1 (Pin_1), U5.15 (TP_SCL)
- new net Screen_VCC: C14.1, C16.1, J8.4 (Pin_4), U5.10 (TP_VDD), U5.3 (BL_A), U5.4 (DP_VDD)
- no-connect marks 40 -> 44
Other:
- note added: "Screen Connector"
- note added: "Screen with touchpad ID: 0010101 0x15"
- note removed: "Screen with touchpad ID:"
- moved on the sheet: C14, C15, C16, C17, C18, C19, C21, J3, R22, R27, RN1, U5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
