File: Module/@ESP32_S2_WROVER_EVB/ESP32_S2_WROVER_EVB.kicad_pcb (KiCad board)
At the start: 4 copper layers, 132.5 x 75 mm, 123 parts, among them J1 CQ-USB-C16PSMT01, J2 microSD, J3 Motor, J4 ADC_IN1, J5 Out BK, J7 Screen_C, J8 Screen_C, Q1 Q_NPN_BEC, Q2 Q_NPN_BEC, SW1 SW_Push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

Commit message: update ESP32_S2_WROVER_EVB
Changed lines of the file:
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@@
     (property "Sheetname" "")
     (attr exclude_from_pos_files)
-    (fp_text reference "H7" (at 0 -4.2) (layer "F.SilkS")
+    (fp_text reference "H7" (at 0 0.07) (layer "F.SilkS")
       (effects (font (size 1 1) (thickness 0.15)))
     )
@@
   )
   (footprint "Package_LGA:Bosch_LGA-14_3x2.5mm_P0.5mm" (layer "B.Cu")
-    (at 170 95 90)
+    (at 169.955094 95 90)
     (descr "LGA-14 Bosch https://ae-bst.resource.bosch.com/media/_tech/media/datasheets/BST-BMI160-DS000-07.pdf")
     (tags "lga land grid array")
@@
   (arc (start 169.310094 61.813726) (mid 169.351677 62.022776) (end 169.470094 62.2) (width 0.2) (layer "F.Cu") (net 1))
   (segment (start 168.942594 95.5) (end 168.005094 95.5) (width 0.2) (layer "B.Cu") (net 1))
+  (segment (start 169.205094 93.404264) (end 169.205094 93.7375) (width 0.15) (layer "B.Cu") (net 1))
   (segment (start 196.070094 131.23) (end 196.070094 130.6) (width 0.2) (layer "B.Cu") (net 1))
   (segment (start 141.755094 90.5) (end 141.755094 91.5) (width 0.4) (layer "B.Cu") (net 1))
+  (segment (start 169.107962 93.182868) (end 169.117226 93.192132) (width 0.15) (layer "B.Cu") (net 1))
   (segment (start 135.980094 93.2) (end 135.980094 92.1375) (width 0.4) (layer "B.Cu") (net 1))
   (segment (start 140.155094 66.4) (end 139.694505 66.860589) (width 0.3) (layer "B.Cu") (net 1))
   (segment (start 205.039998 74.833001) (end 205.04 74.832999) (width 0.15) (layer "B.Cu") (net 1))
-  (segment (start 167.525 93.095) (end 168.990094 93.095) (width 0.2) (layer "B.Cu") (net 1))
   (segment (start 182.000002 68.482998) (end 182.000002 69.23) (width 0.2) (layer "B.Cu") (net 1))
   (segment (start 182.000002 68.482998) (end 182.000002 67.213004) (width 0.2) (layer "B.Cu") (net 1))
@@
   (segment (start 142.655094 91.5) (end 141.745094 91.5) (width 0.4) (layer "B.Cu") (net 1))
   (segment (start 142.355094 90.5) (end 142.355094 91.5) (width 0.4) (layer "B.Cu") (net 1))
-  (segment (start 169.255094 93.36) (end 169.255094 93.732406) (width 0.2) (layer "B.Cu") (net 1))
+  (segment (start 167.525 93.095) (end 168.89583 93.095) (width 0.15) (layer "B.Cu") (net 1))
   (segment (start 171.755094 94.125) (end 171.755094 93.5) (width 0.2) (layer "B.Cu") (net 1))
   (segment (start 136.630094 97.8625) (end 136.630094 99.457495) (width 0.4) (layer "B.Cu") (net 1))
@@
   (segment (start 142.655094 90.5) (end 142.655094 91.5) (width 0.4) (layer "B.Cu") (net 1))
   (segment (start 205.04 74.832999) (end 205.04 72.7) (width 0.2) (layer "B.Cu") (net 1))
-  (arc (start 168.990094 93.095) (mid 169.177477 93.172617) (end 169.255094 93.36) (width 0.2) (layer "B.Cu") (net 1))
+  (arc (start 169.117226 93.192132) (mid 169.182258 93.289459) (end 169.205094 93.404264) (width 0.15) (layer "B.Cu") (net 1))
   (arc (start 171.380094 94.5) (mid 171.645259 94.390165) (end 171.755094 94.125) (width 0.2) (layer "B.Cu") (net 1))
   (arc (start 136.630094 99.457495) (mid 136.578837 99.581241) (end 136.455091 99.632498) (width 0.4) (layer "B.Cu") (net 1))
   (arc (start 182.000002 67.213004) (mid 182.000002 67.213002) (end 182 67.213) (width 0.4) (layer "B.Cu") (net 1))
-  (arc (start 169.255094 93.732406) (mid 169.253602 93.736008) (end 169.25 93.7375) (width 0.2) (layer "B.Cu") (net 1))
   (arc (start 167.530094 94.370094) (mid 167.528602 94.366492) (end 167.525 94.365) (width 0.2) (layer "B.Cu") (net 1))
   (arc (start 171.755094 93.5) (mid 171.872251 93.217157) (end 172.155094 93.1) (width 0.2) (layer "B.Cu") (net 1))
   (arc (start 172.47 93.1) (mid 172.473536 93.098536) (end 172.475 93.095) (width 0.2) (layer "B.Cu") (net 1))
   (arc (start 137.280094 99.457498) (mid 137.33135 99.581242) (end 137.455094 99.632498) (width 0.4) (layer "B.Cu") (net 1))
+  (arc (start 169.107962 93.182868) (mid 169.010635 93.117836) (end 168.89583 93.095) (width 0.15) (layer "B.Cu") (net 1))
   (arc (start 168.005094 95.5) (mid 167.669218 95.360876) (end 167.530094 95.025) (width 0.2) (layer "B.Cu") (net 1))
   (segment (start 179.65 123.79) (end 179.65 124.54) (width 0.2) (layer "F.Cu") (net 2))
@@
   (arc locked (start 189.658694 85.911308) (mid 189.898755 85.552025) (end 189.983056 85.128228) (width 0.2) (layer "F.Cu") (net 111))
   (arc locked (start 189.983056 85.128228) (mid 189.805247 84.234319) (end 189.298891 83.476501) (width 0.2) (layer "F.Cu") (net 111))
-  (segment (start 93.5 78.6) (end 96.75 78.6) (width 0.5) (layer "F.Cu") (net 113))
-  (via (at 96.75 78.6) (size 0.45) (drill 0.2) (layers "F.Cu" "B.Cu") (net 113))
-  (via (at 93.5 78.6) (size 0.45) (drill 0.2) (layers "F.Cu" "B.Cu") (net 113))
+  (segment (start 93.5 78.6) (end 96.75 78.6) (width 0.7) (layer "F.Cu") (net 113))
+  (via (at 96.75 78.6) (size 0.45) (drill 0.3) (layers "F.Cu" "B.Cu") (net 113))
+  (via (at 93.5 78.6) (size 0.45) (drill 0.3) (layers "F.Cu" "B.Cu") (net 113))
   (segment (start 87.735094 88.11) (end 90.851818 84.993276) (width 0.7) (layer "B.Cu") (net 113))
   (segment (start 84.373654 104.926346) (end 83.3 106) (width 0.5) (layer "B.Cu") (net 113))
