File: Module/@ESP32_S2_WROVER_EVB/ESP32_S2_WROVER_EVB.kicad_sch (KiCad schematic)
At the start: 123 parts, among them J1 CQ-USB-C16PSMT01, J2 microSD, J3 Motor, J4 ADC_IN1, J5 Out BK, J7 Screen_C, J8 Screen_C, Q1 Q_NPN_BEC, Q2 Q_NPN_BEC, SW1 SW_Push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

Commit message: update ESP32_S2_WROVER_EVB
Parts:
- H7: value (none) -> Solid; footprint (none) -> MountingHole:MountingHole_3.2mm_M3_Pad_Via
Changed lines of the file:
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@@
       (effects (font (size 1.27 1.27)) (justify left))
     )
-    (property "Value" "" (id 1) (at 201.93 60.1222 0)
+    (property "Value" "Solid" (id 1) (at 201.93 60.1222 0)
       (effects (font (size 1.27 1.27)) (justify left))
     )
-    (property "Footprint" "" (id 2) (at 199.39 59.69 0)
+    (property "Footprint" "MountingHole:MountingHole_3.2mm_M3_Pad_Via" (id 2) (at 199.39 59.69 0)
       (effects (font (size 1.27 1.27)) hide)
     )
